File: pcb/COSV-PCB/Carrier-TEESNSY40/cosv-carrier-teensy40.brd (EAGLE design)
At the start: 96.8 x 26.7 mm, 21 parts, among them K1 61200821621, K2 61200821621, K3 61200821621

Commit message: update teensy carrier board for 12/12 design rules
Routing:
- net 3V3: track 113.3 -> 126.6 mm
- net GND: track 243.6 -> 252.6 mm, vias 0 -> 2
- net A_BATTERY: track 54.6 -> 56.1 mm
- net SDA1: track 18.1 -> 17.0 mm
- net LINE_DETECT: track 29.1 -> 29.9 mm
- removed copper zone on layer 16, net GND
